File: A/A.kicad_pcb (KiCad board)
At the start: 2 copper layers, 582 parts, among them IC1 NCP380 ADJ, J1 Conn_02x06_Top_Bottom, J10 Conn_01x06, J11 DCJ200-10-A-XX-K_REVA, J12 USB_B, J13 Conn_01x08_Pin, J14 Conn_01x02, J15 Conn_01x02, J2 Conn_02x08_Top_Bottom, J3 Conn_01x02, J4 Conn_02x08_Top_Bottom, J5 Conn_01x04, J6 Conn_02x03_Top_Bottom, J7 Conn_01x08, J8 08B0-1X1T-36-F, J9 Conn_01x06, Q1 CSD25310Q2, Q10 DMMT5401-7-F, Q11 DMMT5401-7-F, Q12 DMMT5401-7-F, Q2 BF459, Q3 BF459, Q4 BF459, Q5 BF459, Q6 BF459, Q7 DMMT5401-7-F, Q8 DMMT5401-7-F, Q9 DMMT5401-7-F, SW0 EG1218, SW1 EG1218, SW2 EG1218, SW3 EG1218, U1 XC7A100T-1CSG324C, U11 FT2232HL-REEL, U12 93LC56BT-I_OT, U13 TPD4E101DPWR, U14 SN74LVC126APW, U2 DP83848JSQ_NOPB, U3 MT41K128M16JT-125_K, U4 MP5470GL-0000-Z, U5 MP8756GD-Z, U6 INA199A1DCKR, U7 INA199A1DCKR, U8 REF3012AIDBZR, U9 AP2303MPTR-G1, Y1 25MHz, Y3 25MHz, Y4 ASEM1-100.000MHZ-LC-T, Y5 ASEM1-100.000MHZ-LC-T

Commit message: Add files via upload
Updated
Parts:
- removed C186, C190, C192: 470nF, Capacitor_SMD:C_0805_2012Metric
- removed C187, C191: 47nF, Capacitor_SMD:C_0805_2012Metric
- removed C188: 47uF, Capacitor_SMD:C_0201_0603Metric
- removed C189, C193: 100uF, Capacitor_SMD:C_0805_2012Metric
- removed C202, C203: 100nF, Capacitor_SMD:C_0402_1005Metric
- removed LD0, LD1, LD2, LD3: 19-337/R6GHBHC-A01/2T, 19-337_R6GHBHC-A01_2T:LED_19-337_R6GHBHC-A01_2T
- removed Q5, Q6: BF459, Package_TO_SOT_THT:TO-126-3_Vertical
- removed SW0, SW1, SW2, SW3: EG1218, EG1218:SW_EG1218
- added C60: 47uF, Capacitor_SMD:C_1210_3225Metric, F.Cu at (39.7, 150.0)
- added C61: 470nF, Capacitor_SMD:C_0603_1608Metric, F.Cu at (22.9, 130.8)
- added C62: 4.7uF, Capacitor_SMD:C_0805_2012Metric, F.Cu at (45.7, 126.3)
- added C63: 470nF, Capacitor_SMD:C_0603_1608Metric, F.Cu at (22.9, 133.4)
- added C64: 47nF, Capacitor_SMD:C_1206_3216Metric, F.Cu at (23.7, 104.5)
- added C65: 4.7uF, Capacitor_SMD:C_0805_2012Metric, F.Cu at (45.7, 129.4)
- added C66: 470nF, Capacitor_SMD:C_0603_1608Metric, F.Cu at (22.9, 135.9)
- added C67: 470nF, Capacitor_SMD:C_0603_1608Metric, F.Cu at (22.9, 138.4)
- added C68: 470nF, Capacitor_SMD:C_0603_1608Metric, F.Cu at (22.9, 140.9)
- added C69: 470nF, Capacitor_SMD:C_0603_1608Metric, F.Cu at (22.9, 143.4)
- added C70: 47nF, Capacitor_SMD:C_1206_3216Metric, F.Cu at (23.7, 107.8)
- added D1: 19-337_R6GHBHC-A01_2T, 19-337_R6GHBHC-A01_2T:LED_19-337_R6GHBHC-A01_2T, F.Cu at (129.0, 124.3)
- added D2: 19-337_R6GHBHC-A01_2T, 19-337_R6GHBHC-A01_2T:LED_19-337_R6GHBHC-A01_2T, F.Cu at (135.6, 124.3)
- added D3: 19-337_R6GHBHC-A01_2T, 19-337_R6GHBHC-A01_2T:LED_19-337_R6GHBHC-A01_2T, F.Cu at (142.1, 124.3)
- added D4: 19-337_R6GHBHC-A01_2T, 19-337_R6GHBHC-A01_2T:LED_19-337_R6GHBHC-A01_2T, F.Cu at (148.7, 124.3)
- added D5: D_TVS, Diode_SMD:D_0603_1608Metric, F.Cu at (278.3, 227.2)
- added D6: D_TVS, Diode_SMD:D_0603_1608Metric, F.Cu at (278.3, 229.8)
- added JP2: Conn_01x02, Connector_PinHeader_1.00mm:PinHeader_1x02_P1.00mm_Vertical, F.Cu at (225.6, 67.5)
- added R123: 100E, Resistor_SMD:R_0402_1005Metric, F.Cu at (27.4, 72.8)
- added S1: EG1218, EG1218:SW_EG1218, F.Cu at (156.3, 120.3)
- added S2: EG1218, EG1218:SW_EG1218, F.Cu at (162.9, 120.4)
- added S3: EG1218, EG1218:SW_EG1218, F.Cu at (169.8, 120.3)
- added S4: EG1218, EG1218:SW_EG1218, F.Cu at (176.6, 120.4)
- added U10: S25FL128SAGMFI013, ul_S25FL128SAGMFI013:SO3016_SPA, F.Cu at (160.0, 71.0)
- C100, C102: value 470uF -> 470nF; footprint Capacitor_SMD:C_1812_4532Metric -> Capacitor_SMD:C_0603_1608Metric
- C105: footprint Capacitor_SMD:C_0402_1005Metric -> Capacitor_SMD:C_0603_1608Metric_Pad1.08x0.95mm_HandSolder
- C109: footprint Capacitor_SMD:C_1206_3216Metric -> Capacitor_SMD:C_0402_1005Metric
- C113, C136, C137, C138, C145, C146, C147, C153, C159, C167: value 100uF -> 47nF; footprint Capacitor_SMD:C_0805_2012Metric -> Capacitor_SMD:C_1206_3216Metric
- C114, C123, C124: value 4.7uF -> 47nF; footprint Capacitor_SMD:C_0402_1005Metric -> Capacitor_SMD:C_1206_3216Metric
- C115, C172, C173: footprint Capacitor_SMD:C_0402_1005Metric -> Capacitor_SMD:C_0805_2012Metric
- C116: value 470nF -> 100uF; footprint Capacitor_SMD:C_0805_2012Metric -> Capacitor_SMD:C_1206_3216Metric
- C117, C118: value 470nF -> 4.7uF
- C119, C176, C177, C184: footprint Capacitor_SMD:C_0805_2012Metric -> Capacitor_SMD:C_0603_1608Metric
- C120, C121, C122: value 47nF -> 470nF; footprint Capacitor_SMD:C_0805_2012Metric -> Capacitor_SMD:C_0603_1608Metric
- C125: value 470nF -> 47nF; footprint Capacitor_SMD:C_0805_2012Metric -> Capacitor_SMD:C_1206_3216Metric
- C126, C127, C128: value 470nF -> 10nF; footprint Capacitor_SMD:C_0805_2012Metric -> Capacitor_SMD:C_0201_0603Metric
- C129: value 47nF -> 100uF; footprint Capacitor_SMD:C_0805_2012Metric -> Capacitor_SMD:C_1206_3216Metric
- C130, C131: value 47nF -> 4.7uF
- C132, C133, C134, C135, C141, C142, C143, C144, C151, C152, C163, C164, C165, C166: value 100uF -> 470nF; footprint Capacitor_SMD:C_0805_2012Metric -> Capacitor_SMD:C_0603_1608Metric
- C139, C140, C149, C150, C161, C162, C170, C171: value 100uF -> 4.7uF
- C14, C15, C16, C17, C18, C19: footprint Capacitor_SMD:C_1206_3216Metric -> Capacitor_SMD:C_0805_2012Metric
- C148, C168, C169, C20, C21, C22, C24, C25, C26, C28, C29, C30, C32, C33, C35, C36, C38, C39, C41, C42, C44, C45: footprint Capacitor_SMD:C_0805_2012Metric -> Capacitor_SMD:C_1206_3216Metric
- C154, C156, C157, C158: value 100nF -> 47nF; footprint Capacitor_SMD:C_0402_1005Metric -> Capacitor_SMD:C_1206_3216Metric
- C155: value 100nF -> 470nF; footprint Capacitor_SMD:C_0402_1005Metric -> Capacitor_SMD:C_0603_1608Metric
- C160: value 100uF -> 47uF; footprint Capacitor_SMD:C_0805_2012Metric -> Capacitor_SMD:C_1210_3225Metric
- C174, C175, C182: value 4.7uF -> 470nF; footprint Capacitor_SMD:C_0402_1005Metric -> Capacitor_SMD:C_0603_1608Metric
- C178: value 470uF -> 470nF; footprint Capacitor_SMD:C_0805_2012Metric -> Capacitor_SMD:C_0603_1608Metric
- C179: value 470uF -> 10nF; footprint Capacitor_SMD:C_0805_2012Metric -> Capacitor_SMD:C_0201_0603Metric
- C180: value 470uF -> 100nF; footprint Capacitor_SMD:C_0805_2012Metric -> Capacitor_SMD:C_0201_0603Metric
- C181: value 4.7uF -> 100uF; footprint Capacitor_SMD:C_0402_1005Metric -> Capacitor_SMD:C_1206_3216Metric
- C183: value 470uF -> 47nF; footprint Capacitor_SMD:C_0805_2012Metric -> Capacitor_SMD:C_1206_3216Metric
- C185: value 470nF -> 100nF
- C83, C84, C85, C88, C89: footprint Capacitor_SMD:C_0201_0603Metric -> Capacitor_SMD:C_0402_1005Metric
- J1: value Conn_02x06_Top_Bottom -> Conn_02x06_Odd_Even
- J12: footprint Connector_USB:USB_B_TE_5787834_Vertical -> Connector_USB:USB_Micro-B_Amphenol_10103594-0001LF_Horizontal
- J2, J4: value Conn_02x08_Top_Bottom -> Conn_02x08_Odd_Even
- J6: value Conn_02x03_Top_Bottom -> Conn_02x03_Odd_Even; footprint Connector_PinHeader_2.54mm:PinHeader_2x03_P2.54mm_Vertical -> Connector_PinSocket_2.54mm:PinSocket_2x03_P2.54mm_Vertical
- Q3, Q4: value BF459 -> DMMT5401-7-F; footprint Package_TO_SOT_THT:TO-126-3_Vertical -> DMMT5401-7-F:SOT95P285X140-6N
- R1, R10, R100, R101, R102, R103, R104, R105, R106, R107, R108, R109, R11, R129, R132, R136, R155, R156, R158, R167, R168, R169, R172, R178, R179, R18, R180, R181, R182, R183, R186, R187, R188, R189, R19, R190, R191, R195, R196, R197, R198, R199, R2, R200, R204, R205, R206, R207, R208, R209, R22, R248, R249, R3, R4, R5, R59, R6, R60, R61, R62, R63, R64, R65, R66, R67, R68, R69, R70, R71, R73, R75, R77, R79, R8, R81, R83, R84, R85, R86, R87, R88, R89, R9, R90, R91, R92, R93, R94, R95, R96, R98, R99: footprint Resistor_SMD:R_0201_0603Metric -> Resistor_SMD:R_0402_1005Metric
- R111, R112, R113, R114, R115, R116, R117, R118, R119, R120, R121, R122, R125, R138, R17, R21, R23, R24, R251, R252, R255, R256, R257, R277, R278, R279, R280, R281, R282, R283, R284, R285, R286, R287, R288, R289, R290, R291, R292, R293, R294, R298, R299, R300, R301, R302, R303, R304, R305, R306, R307, R308, R72, R74, R76, R78, R80, R82: footprint Resistor_SMD:R_1206_3216Metric -> Resistor_SMD:R_0402_1005Metric
- R12, R13, R131, R135, R14, R140, R157, R160, R162, R163, R164, R165, R170, R171, R246, R247, R25, R26, R261, R262, R263, R264, R265, R266, R267, R268, R27, R28, R29, R30, R31, R32, R33, R34, R35, R36, R7, R97: footprint Resistor_SMD:R_0805_2012Metric -> Resistor_SMD:R_0402_1005Metric
- R166, R175, R192, R201: value 86.6 -> 86.6E; footprint Resistor_SMD:R_0201_0603Metric -> Resistor_SMD:R_0402_1005Metric
- R173, R174, R37, R38: value 330 -> 330E; footprint Resistor_SMD:R_0201_0603Metric -> Resistor_SMD:R_0402_1005Metric
- R176, R184, R193, R202: value 150 -> 150E; footprint Resistor_SMD:R_2512_6332Metric -> Resistor_SMD:R_0402_1005Metric
- R177, R185, R194, R203: value 75 -> 75E; footprint Resistor_SMD:R_0805_2012Metric -> Resistor_SMD:R_0402_1005Metric
- R250, R253, R254, R271, R272, R273, R274, R275, R276, R296, R297: footprint Resistor_SMD:R_0603_1608Metric -> Resistor_SMD:R_0402_1005Metric
- R259: value 100 -> 100E
- moved R225 277.8 mm to (377.9, 23.5)
- moved R216 277.6 mm to (375.0, 23.5)
- moved R217 277.6 mm to (375.0, 25.4)
- moved R234 273.7 mm to (380.8, 23.5)
- moved R235 273.7 mm to (380.8, 25.4)
- moved R236 273.7 mm to (380.8, 27.4)
- moved R237 273.7 mm to (380.8, 29.4)
- moved R238 273.7 mm to (380.8, 31.4)
- moved R239 273.7 mm to (380.8, 33.4)
- moved R240 273.7 mm to (380.8, 35.4)
- moved R241 273.7 mm to (380.8, 37.4)
- moved R226 273.6 mm to (377.9, 25.4)
- moved R227 273.6 mm to (377.9, 27.4)
- moved R228 273.6 mm to (377.9, 29.4)
- moved R229 273.6 mm to (377.9, 31.4)
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Connections:
- net Net-(J6-Pin_1) renamed /CHIPKIT IO/MISO
- net SW0 renamed S1
- net SW1 renamed S2
- net SW2 renamed S3
- net SW3 renamed S4
- BTN0 pad 1: A17 -> +3V3
- BTN0 pad 2: A17 -> +3V3
- BTN1 pad 1: A17 -> +3V3
- BTN1 pad 2: A17 -> +3V3
- BTN2 pad 1: A17 -> +3V3
- BTN2 pad 2: A17 -> +3V3
- BTN3 pad 1: A17 -> +3V3
- BTN3 pad 2: A17 -> +3V3
- BTN4 pad 3: A17 -> GND
- BTN4 pad 4: A17 -> GND
- BTN5 pad 1: A17 -> GND
- BTN5 pad 2: A17 -> GND
- C1 pad 1: A17 -> +3V3
- C1 pad 2: A17 -> GND
- C10 pad 2: A17 -> GND
- C100 pad 2: A17 -> GND
- C101 pad 2: A17 -> GND
- C102 pad 2: A17 -> GND
- C103 pad 2: A17 -> GND
- C109 pad 1: A17 -> +3V3
- C109 pad 2: A17 -> GND
- C11 pad 2: A17 -> GND
- C113 pad 1: A17 -> +3V3
- C113 pad 2: A17 -> GND
- C114 pad 1: A17 -> +3V3
- C114 pad 2: A17 -> GND
- C115 pad 1: A17 -> +3V3
- C115 pad 2: A17 -> GND
- C116 pad 1: A17 -> DDRVCC
- C116 pad 2: A17 -> GND
- C117 pad 1: A17 -> DDRVCC
- C117 pad 2: A17 -> GND
- C118 pad 1: A17 -> DDRVCC
- C118 pad 2: A17 -> GND
- C119 pad 1: A17 -> DDRVCC
- C119 pad 2: A17 -> GND
- C12 pad 2: A17 -> GND
- C120 pad 1: A17 -> DDRVCC
- C120 pad 2: A17 -> GND
- C121 pad 1: A17 -> DDRVCC
- C121 pad 2: A17 -> GND
- C122 pad 1: A17 -> DDRVCC
- C122 pad 2: A17 -> GND
- C123 pad 1: A17 -> DDRVCC
- C123 pad 2: A17 -> GND
- C124 pad 1: A17 -> DDRVCC
- C124 pad 2: A17 -> GND
- C125 pad 1: A17 -> DDRVCC
- C125 pad 2: A17 -> GND
- C126 pad 1: A17 -> DDRVCC
- C126 pad 2: A17 -> GND
- C127 pad 1: A17 -> DDRVCC
- C127 pad 2: A17 -> GND
- C128 pad 1: A17 -> DDRVCC
- C128 pad 2: A17 -> GND
- C129 pad 1: A17 -> +3V3
- C129 pad 2: A17 -> GND
- C13 pad 2: A17 -> GND
- C130 pad 1: A17 -> +3V3
- C130 pad 2: A17 -> GND
- C131 pad 1: A17 -> +3V3
- C131 pad 2: A17 -> GND
- C132 pad 1: A17 -> +3V3
- C132 pad 2: A17 -> GND
- C133 pad 1: A17 -> +3V3
- C133 pad 2: A17 -> GND
- C134 pad 1: A17 -> +3V3
- C134 pad 2: A17 -> GND
- C135 pad 1: A17 -> +3V3
- C135 pad 2: A17 -> GND
- C136 pad 1: A17 -> +3V3
- C136 pad 2: A17 -> GND
- C137 pad 1: A17 -> +3V3
- C137 pad 2: A17 -> GND
- C138 pad 1: A17 -> +3V3
- C138 pad 2: A17 -> GND
- C139 pad 1: A17 -> +3V3
- C139 pad 2: A17 -> GND
- C140 pad 1: A17 -> +3V3
- C140 pad 2: A17 -> GND
- C141 pad 1: A17 -> +3V3
- C141 pad 2: A17 -> GND
- C142 pad 1: A17 -> +3V3
- C142 pad 2: A17 -> GND
- C143 pad 1: A17 -> +3V3
- C143 pad 2: A17 -> GND
- C144 pad 1: A17 -> +3V3
- C144 pad 2: A17 -> GND
- C145 pad 1: A17 -> +3V3
- C145 pad 2: A17 -> GND
- C146 pad 1: A17 -> +3V3
- C146 pad 2: A17 -> GND
- C147 pad 1: A17 -> +3V3
- C147 pad 2: A17 -> GND
- C148 pad 1: A17 -> +1V0
- C148 pad 2: A17 -> GND
- C149 pad 1: A17 -> +1V0
- C149 pad 2: A17 -> GND
- C150 pad 1: A17 -> +1V0
- C150 pad 2: A17 -> GND
- C151 pad 1: A17 -> +1V0
- C151 pad 2: A17 -> GND
- C152 pad 1: A17 -> +1V0
- C152 pad 2: A17 -> GND
- C153 pad 1: A17 -> +1V0
- C153 pad 2: A17 -> GND
- C154 pad 1: A17 -> +1V0
- C154 pad 2: A17 -> GND
- C155 pad 1: A17 -> +1V0
- C155 pad 2: A17 -> GND
- C156 pad 1: A17 -> +1V0
- C156 pad 2: A17 -> GND
- C157 pad 1: A17 -> +1V0
- C157 pad 2: A17 -> GND
- C158 pad 1: A17 -> +1V0
- C158 pad 2: A17 -> GND
- C159 pad 1: A17 -> +1V0
- C159 pad 2: A17 -> GND
- C160 pad 1: A17 -> +1V8
- C160 pad 2: A17 -> GND
- C161 pad 1: A17 -> +1V8
- C161 pad 2: A17 -> GND
- C162 pad 1: A17 -> +1V8
- C162 pad 2: A17 -> GND
- C163 pad 1: A17 -> +1V8
- C163 pad 2: A17 -> GND
- C164 pad 1: A17 -> +1V8
- C164 pad 2: A17 -> GND
- C165 pad 1: A17 -> +1V8
- C165 pad 2: A17 -> GND
- C166 pad 1: A17 -> +1V8
- C166 pad 2: A17 -> GND
- C167 pad 1: A17 -> +1V8
- C167 pad 2: A17 -> GND
- C168 pad 1: A17 -> +1V0
- C168 pad 2: A17 -> GND
- C169 pad 1: A17 -> +1V0
- C169 pad 2: A17 -> GND
- C170 pad 1: A17 -> +1V0
- C170 pad 2: A17 -> GND
- C171 pad 1: A17 -> +1V0
- C171 pad 2: A17 -> GND
- C172 pad 1: A17 -> +1V0
- C172 pad 2: A17 -> GND
- C173 pad 1: A17 -> +1V0
- C173 pad 2: A17 -> GND
- C174 pad 1: A17 -> +1V0
- C174 pad 2: A17 -> GND
- C175 pad 1: A17 -> +1V0
- C175 pad 2: A17 -> GND
- C176 pad 1: A17 -> +1V0
- C176 pad 2: A17 -> GND
- C177 pad 1: A17 -> +1V0
- C177 pad 2: A17 -> GND
- C178 pad 1: A17 -> +1V0
- C178 pad 2: A17 -> GND
- C179 pad 1: A17 -> +1V8
- C179 pad 2: A17 -> GND
- C180 pad 1: A17 -> +1V8
- C180 pad 2: A17 -> GND
- C181 pad 1: F10 -> +1V0
- C181 pad 2: A17 -> GND
- C182 pad 1: F10 -> +1V0
- C182 pad 2: A17 -> GND
- C183 pad 1: F10 -> +1V0
- C183 pad 2: A17 -> GND
- C184 pad 1: F10 -> +1V0
- C184 pad 2: A17 -> GND
- C185 pad 1: F10 -> +3V3
- C185 pad 2: A17 -> CK_RST
- C194 pad 1: A17 -> GND
- C194 pad 2: A17 -> +3V3
- C195 pad 2: A17 -> GND
- C196 pad 2: A17 -> GND
- C197 pad 2: A17 -> GND
- C198 pad 2: A17 -> GND
- C199 pad 2: A17 -> GND
- C2 pad 1: A17 -> +3V3
- C2 pad 2: A17 -> GND
- C20 pad 2: A17 -> GND
- C200 pad 2: A17 -> GND
- C201 pad 1: A17 -> +3V3
- C201 pad 2: A17 -> GND
- C204 pad 1: A17 -> +3V3
- C204 pad 2: A17 -> GND
- C21 pad 2: A17 -> GND
- C22 pad 2: A17 -> GND
- C23 pad 2: A17 -> GND
- C24 pad 2: A17 -> GND
- C25 pad 2: A17 -> GND
- C26 pad 2: A17 -> GND
- C27 pad 2: A17 -> GND
- C28 pad 2: A17 -> GND
- C29 pad 2: A17 -> GND
- C3 pad 1: A17 -> +3V3
- C3 pad 2: A17 -> GND
- C30 pad 2: A17 -> GND
- C31 pad 2: A17 -> GND
- C32 pad 2: A17 -> GND
- C33 pad 2: A17 -> GND
- C34 pad 2: A17 -> GND
- C35 pad 2: A17 -> GND
- C36 pad 2: A17 -> GND
- C37 pad 2: A17 -> GND
- C38 pad 2: A17 -> GND
- C39 pad 2: A17 -> GND
- C4 pad 1: A17 -> +3V3
- C4 pad 2: A17 -> GND
- C40 pad 2: A17 -> GND
- C41 pad 2: A17 -> GND
- C42 pad 2: A17 -> GND
- C43 pad 2: A17 -> GND
- C44 pad 2: A17 -> GND
- C45 pad 2: A17 -> GND
- C46 pad 2: A17 -> GND
- C47 pad 2: A17 -> GND
- C48 pad 2: A17 -> GND
- C5 pad 2: A17 -> GND
- C50 pad 2: A17 -> GND
- C51 pad 2: A17 -> GND
- C52 pad 2: A17 -> GND
- C53 pad 1: F10 -> +1V8
- C53 pad 2: A17 -> GND
- C54 pad 1: A17 -> +3V3
- C54 pad 2: A17 -> GND
- C55 pad 2: A17 -> GND
- C56 pad 2: A17 -> GND
- C57 pad 2: A17 -> GND
- C58 pad 2: A17 -> GND
- C59 pad 2: A17 -> GND
- C6 pad 2: A17 -> GND
- C7 pad 2: A17 -> GND
- C71 pad 1: A17 -> GND
- C72 pad 1: A17 -> GND
- C73 pad 1: A17 -> GND
- C74 pad 1: F10 -> XADCGND
- C75 pad 1: A17 -> GND
- C76 pad 1: A17 -> GND
- C77 pad 1: A17 -> GND
- C79 pad 1: F10 -> XADCGND
- C8 pad 2: A17 -> GND
- C81 pad 1: A17 -> GND
- C82 pad 1: A17 -> GND
- C83 pad 2: A17 -> GND
- C84 pad 2: A17 -> GND
- C85 pad 2: A17 -> GND
- C86 pad 2: A17 -> GND
- C87 pad 2: A17 -> GND
- C88 pad 2: A17 -> GND
- C89 pad 2: A17 -> GND
- C9 pad 2: A17 -> GND
- C90 pad 2: A17 -> GND
- C91 pad 2: A17 -> GND
- C92 pad 2: A17 -> GND
- C93 pad 2: A17 -> GND
- C94 pad 2: A17 -> GND
- C95 pad 2: A17 -> GND
- C96 pad 2: A17 -> GND
- C97 pad 2: A17 -> GND
- C98 pad 1: A17 -> +3V3
- C98 pad 2: A17 -> GND
- C99 pad 2: A17 -> GND
- FB1 pad 1: A17 -> GND
- FB1 pad 2: F10 -> XADCGND
- FB3 pad 1: A17 -> +3V3
- FB4 pad 1: A17 -> +3V3
- FB5 pad 1: A17 -> +3V3
- FB6 pad 1: A17 -> GND
- FB6 pad 2: A17 -> GND
- FB8 pad 1: A17 -> GND
- J1 pad 10: CK_A9 -> CK_A10
- J1 pad 11: CK_A10 -> CK_A5
- J1 pad 2: CK_A1 -> CK_A6
- J1 pad 3: CK_A2 -> CK_A1
- J1 pad 4: CK_A3 -> CK_A7
- J1 pad 5: CK_A4 -> CK_A2
- J1 pad 6: CK_A5 -> CK_A8
- J1 pad 7: CK_A6 -> CK_A3
- J1 pad 8: CK_A7 -> CK_A9
- J1 pad 9: CK_A8 -> CK_A4
- J10 pad 5: A17 -> GND
- J10 pad 6: A17 -> +3V3
- J11 pad 2: A17 -> GND
- J11 pad 3: A17 -> GND
- J13 pad 1: A17 -> +3V3
- J13 pad 8: A17 -> GND
- J14 pad 1: A17 -> +3V3
- J14 pad 2: A17 -> GND
- J15 pad 1: A17 -> +3V3
- J15 pad 2: A17 -> GND
- J2 pad 10: /CHIPKIT IO/35 -> /CHIPKIT IO/38
- J2 pad 11: /CHIPKIT IO/36 -> /CHIPKIT IO/13
- J2 pad 12: /CHIPKIT IO/37 -> /CHIPKIT IO/39
- J2 pad 13: /CHIPKIT IO/38 -> /CHIPKIT IO/G
- J2 pad 14: /CHIPKIT IO/39 -> /CHIPKIT IO/40
- J2 pad 15: /CHIPKIT IO/40 -> /CHIPKIT IO/A
- J2 pad 2: /CHIPKIT IO/9 -> /CHIPKIT IO/34
- J2 pad 3: /CHIPKIT IO/10 -> /CHIPKIT IO/9
- J2 pad 4: /CHIPKIT IO/11 -> /CHIPKIT IO/35
- J2 pad 5: /CHIPKIT IO/12 -> /CHIPKIT IO/10
- J2 pad 6: /CHIPKIT IO/13 -> /CHIPKIT IO/36
- J2 pad 7: /CHIPKIT IO/14 -> /CHIPKIT IO/11
- J2 pad 8: /CHIPKIT IO/15 -> /CHIPKIT IO/37
- J2 pad 9: /CHIPKIT IO/34 -> /CHIPKIT IO/12
- J4 pad 10: /CHIPKIT IO/27 -> /CHIPKIT IO/30
- J4 pad 11: /CHIPKIT IO/28 -> /CHIPKIT IO/5
- J4 pad 12: /CHIPKIT IO/29 -> /CHIPKIT IO/31
- J4 pad 13: /CHIPKIT IO/30 -> /CHIPKIT IO/6
- J4 pad 14: /CHIPKIT IO/31 -> /CHIPKIT IO/32
- J4 pad 15: /CHIPKIT IO/32 -> /CHIPKIT IO/7
- J4 pad 2: /CHIPKIT IO/1 -> /CHIPKIT IO/26
- J4 pad 3: /CHIPKIT IO/2 -> /CHIPKIT IO/1
- J4 pad 4: /CHIPKIT IO/3 -> /CHIPKIT IO/27
- J4 pad 5: /CHIPKIT IO/4 -> /CHIPKIT IO/2
- J4 pad 6: /CHIPKIT IO/5 -> /CHIPKIT IO/28
- J4 pad 7: /CHIPKIT IO/6 -> /CHIPKIT IO/3
- J4 pad 8: /CHIPKIT IO/7 -> /CHIPKIT IO/29
- J4 pad 9: /CHIPKIT IO/26 -> /CHIPKIT IO/4
- J5 pad 3: F10 -> XADCGND
- J6 pad 2: Net-(J6-Pin_2) -> unconnected-(J6-Pin_2-Pad2)
- J6 pad 3: Net-(J6-Pin_3) -> /CHIPKIT IO/SCK
- J6 pad 4: unconnected-(J6-Pin_4-Pad4) -> /CHIPKIT IO/MOSI
- J6 pad 5: Net-(J6-Pin_5) -> /CHIPKIT IO/SS
- J6 pad 6: A17 -> GND
- J7 pad 2: A17 -> +3V3
- J7 pad 4: A17 -> +3V3
- J7 pad 6: A17 -> GND
- J7 pad 7: A17 -> GND
- J9 pad 5: A17 -> GND
- JA1 pad 11: A17 -> GND
- JA1 pad 12: A17 -> +3V3
- JA1 pad 5: A17 -> GND
- JA1 pad 6: A17 -> +3V3
- JB1 pad 11: A17 -> GND
- JB1 pad 12: A17 -> +3V3
- JB1 pad 5: A17 -> GND
- JB1 pad 6: A17 -> +3V3
- JC1 pad 11: A17 -> GND
- JC1 pad 12: A17 -> +3V3
- JC1 pad 5: A17 -> GND
- JC1 pad 6: A17 -> +3V3
- JD1 pad 11: A17 -> GND
- JD1 pad 12: A17 -> +3V3
- JD1 pad 5: A17 -> GND
- JD1 pad 6: A17 -> +3V3
- JP1 pad 2: A17 -> GND
- L3 pad 2: F10 -> +1V8
- L4 pad 2: A17 -> +3V3
- LD4 pad 1: A17 -> GND
- LD5 pad 1: A17 -> GND
- LD6 pad 1: A17 -> GND
- LD7 pad 1: A17 -> GND
- LD8 pad 1: A17 -> GND
- Q10 pad 5: A17 -> GND
- Q10 pad 6: A17 -> GND
- Q11 pad 5: A17 -> GND
- Q11 pad 6: A17 -> GND
- Q12 pad 5: A17 -> GND
- Q12 pad 6: A17 -> GND
- Q3 pad 1: Net-(Q3-E) -> Net-(Q3-Pad1)
- Q3 pad 2: A17 -> Net-(Q3-Pad2)
- Q3 pad 3: Net-(Q3-B) -> Net-(Q3-Pad1)
- Q4 pad 1: Net-(Q3-B) -> GND
- Q4 pad 2: A17 -> PGVREG5V0
- Q4 pad 3: Net-(Q4-B) -> PGVREG5V0
- Q7 pad 5: A17 -> GND
- Q7 pad 6: A17 -> GND
- Q8 pad 5: A17 -> GND
- Q8 pad 6: A17 -> GND
- Q9 pad 5: A17 -> GND
- Q9 pad 6: A17 -> GND
- R1 pad 1: A17 -> +3V3
- R106 pad 1: A17 -> GND
- R121 pad 1: A17 -> GND
- R122 pad 1: A17 -> GND
- R126 pad 1: A17 -> GND
- R127 pad 1: A17 -> GND
- R132 pad 2: A17 -> GND
- R136 pad 2: A17 -> GND
- R138 pad 2: A17 -> GND
- R14 pad 2: A17 -> GND
- R158 pad 2: A17 -> GND
- R161 pad 1: Net-(Q6-C) -> Net-(Q4-Pad6)
- R164 pad 2: A17 -> GND
- R165 pad 2: Net-(Q5-C) -> Net-(Q4-Pad5)
- R167 pad 1: Net-(Q5-C) -> Net-(Q4-Pad5)
- R171 pad 1: Net-(Q3-E) -> Net-(Q3-Pad4)
- R172 pad 1: Net-(Q3-B) -> Net-(Q3-Pad1)
- R18 pad 1: A17 -> GND
- R181 pad 1: A17 -> GND
- R182 pad 1: A17 -> GND
- R183 pad 1: A17 -> GND
- R189 pad 1: A17 -> GND
- R19 pad 1: Net-(Q4-B) -> Net-(Q3-Pad2)
- R190 pad 1: A17 -> GND
- R191 pad 1: A17 -> GND
- R198 pad 1: A17 -> GND
- R199 pad 1: A17 -> GND
- R2 pad 1: A17 -> GND
- R200 pad 1: A17 -> GND
- R207 pad 1: A17 -> GND
- R208 pad 1: A17 -> GND
- R209 pad 1: A17 -> GND
- R24 pad 2: A17 -> GND
- R242 pad 1: A17 -> +3V3
- R243 pad 1: A17 -> +3V3
- R244 pad 1: A17 -> +3V3
- R245 pad 1: A17 -> +3V3
- R246 pad 1: A17 -> +3V3
- R247 pad 1: A17 -> +3V3
- R248 pad 2: A17 -> GND
- R25 pad 1: A17 -> GND
- R251 pad 2: A17 -> +3V3
- R252 pad 2: A17 -> +3V3
- R255 pad 2: A17 -> +3V3
- R256 pad 1: A17 -> GND
- R26 pad 1: A17 -> GND
- R264 pad 2: SNS5V0_P -> SNS5V0_N
- R267 pad 2: SNSVCCINT_P -> SNS5V0_P
- R268 pad 2: SNSVCCINT_N -> SNS5V0_N
- R27 pad 1: A17 -> GND
- R270 pad 2: A17 -> +3V3
- R278 pad 2: A17 -> +3V3
- R279 pad 2: A17 -> +3V3
- R28 pad 1: A17 -> GND
- R280 pad 2: A17 -> +3V3
- R281 pad 1: A17 -> GND
- R282 pad 2: A17 -> +3V3
- R293 pad 1: A17 -> GND
- R3 pad 1: A17 -> GND
- R308 pad 1: A17 -> GND
- R4 pad 1: A17 -> GND
- R40 pad 2: Net-(J6-Pin_2) -> /CHIPKIT IO/SCK
- R41 pad 2: Net-(J6-Pin_3) -> /CHIPKIT IO/SS
- R48 pad 1: A17 -> GND
- R48 pad 2: /CHIPKIT IO/14 -> /CHIPKIT IO/G
- R49 pad 2: /CHIPKIT IO/15 -> /CHIPKIT IO/A
- R5 pad 1: A17 -> +3V3
- R50 pad 1: Net-(J6-Pin_5) -> /CHIPKIT IO/MOSI
- R6 pad 1: A17 -> +3V3
- R60 pad 2: A17 -> GND
- R62 pad 2: A17 -> GND
- R64 pad 2: A17 -> GND
- R66 pad 2: A17 -> GND
- R68 pad 2: A17 -> GND
- R7 pad 1: A17 -> +3V3
- R70 pad 2: A17 -> GND
- R72 pad 2: A17 -> GND
- R74 pad 2: A17 -> GND
- R76 pad 2: A17 -> GND
- R78 pad 2: A17 -> GND
- R80 pad 2: A17 -> GND
- R82 pad 2: A17 -> GND
- R97 pad 2: A17 -> GND
- U1 pad A12: A17 -> GND
- U1 pad A17: A17 -> +3V3
- U1 pad A2: A17 -> GND
- U1 pad A7: A17 -> +3V3
- U1 pad B10: A17 -> +3V3
- U1 pad B15: A17 -> GND
- U1 pad B5: A17 -> GND
- U1 pad C13: A17 -> +3V3
- U1 pad C18: A17 -> GND
- U1 pad C3: A17 -> +3V3
- U1 pad C8: A17 -> GND
- U1 pad D1: A17 -> GND
- U1 pad D11: A17 -> GND
- U1 pad D16: A17 -> +3V3
- U1 pad D6: A17 -> +3V3
- U1 pad E14: A17 -> GND
- U1 pad E4: A17 -> GND
- U1 pad E8: F10 -> +1V8
- U1 pad F11: A17 -> GND
- U1 pad F12: F10 -> +1V8
- U1 pad F17: A17 -> GND
- U1 pad F2: A17 -> +3V3
- U1 pad F7: A17 -> GND
- U1 pad F9: A17 -> GND
- U1 pad G10: A17 -> GND
- U1 pad G12: A17 -> GND
- U1 pad G15: A17 -> +3V3
- U1 pad G5: A17 -> +3V3
- U1 pad G8: A17 -> GND
- U1 pad H11: A17 -> GND
- U1 pad H12: F10 -> +1V8
- U1 pad H13: A17 -> GND
- U1 pad H18: A17 -> +3V3
- U1 pad H3: A17 -> GND
- U1 pad H7: A17 -> GND
- U1 pad H9: A17 -> GND
- U1 pad J1: A17 -> +3V3
- U1 pad J12: A17 -> GND
- U1 pad J16: A17 -> GND
- U1 pad J6: A17 -> GND
- U1 pad J8: A17 -> GND
- U1 pad K11: A17 -> GND
- U1 pad K12: F10 -> +1V8
- U1 pad K14: A17 -> +3V3
- U1 pad K4: A17 -> +3V3
- U1 pad K7: A17 -> GND
- U1 pad L10: A17 -> GND
- U1 pad L12: A17 -> GND
- U1 pad L17: A17 -> +3V3
- U1 pad L2: A17 -> GND
- U1 pad L8: A17 -> GND
- U1 pad L9: A17 -> GND
- U1 pad M11: A17 -> GND
- U1 pad M12: F10 -> +1V8
- U1 pad M15: A17 -> GND
- U1 pad M5: A17 -> GND
- U1 pad M7: A17 -> GND
- U1 pad M9: A17 -> GND
- U1 pad N10: A17 -> GND
- U1 pad N12: A17 -> GND
- U1 pad N13: A17 -> +3V3
- U1 pad N18: A17 -> GND
- U1 pad N3: A17 -> +3V3
- U1 pad N8: A17 -> GND
- U1 pad P1: A17 -> GND
- U1 pad P16: A17 -> +3V3
- U1 pad P6: A17 -> DDRVCC
- U1 pad P8: A17 -> +3V3
- U1 pad R14: A17 -> GND
- U1 pad R4: A17 -> GND
- U1 pad R9: A17 -> +3V3
- U1 pad T12: A17 -> +3V3
- U1 pad T17: A17 -> GND
- U1 pad T2: A17 -> DDRVCC
- U1 pad T7: A17 -> GND
- U1 pad U10: A17 -> GND
- U1 pad U15: A17 -> +3V3
- U1 pad U5: A17 -> DDRVCC
- U1 pad V13: A17 -> GND
- U1 pad V18: A17 -> +3V3
- U1 pad V3: A17 -> GND
- U1 pad V8: A17 -> DDRVCC
- U11 pad 1: A17 -> GND
- U11 pad 10: A17 -> GND
- U11 pad 11: A17 -> GND
- U11 pad 13: A17 -> GND
- U11 pad 15: A17 -> GND
- U11 pad 20: A17 -> +3V3
- U11 pad 25: A17 -> GND
- U11 pad 31: A17 -> +3V3
- U11 pad 35: A17 -> GND
- U11 pad 42: A17 -> +3V3
- U11 pad 47: A17 -> GND
- U11 pad 49: A17 -> +3V3
- U11 pad 5: A17 -> GND
- U11 pad 50: A17 -> GND
- U11 pad 51: A17 -> GND
- U11 pad 56: A17 -> +3V3
- U12 pad 2: A17 -> GND
- U12 pad 6: A17 -> +3V3
- U13 pad 5: A17 -> GND
- U14 pad 7: A17 -> GND
- U2 pad 1: A17 -> +3V3
- U2 pad 13: A17 -> GND
- U2 pad 17: A17 -> GND
- U2 pad 26: A17 -> +3V3
- U2 pad 29: A17 -> GND
- U2 pad 40: A17 -> GND
- U3 pad A9: A17 -> GND
- U3 pad B1: A17 -> GND
- U3 pad B3: A17 -> GND
- U3 pad B9: A17 -> GND
- U3 pad D1: A17 -> GND
- U3 pad D8: A17 -> GND
- U3 pad E1: A17 -> GND
- U3 pad E2: A17 -> GND
- U3 pad E8: A17 -> GND
- U3 pad F9: A17 -> GND
- U3 pad G1: A17 -> GND
- U3 pad G8: A17 -> GND
- U3 pad G9: A17 -> GND
- U3 pad J2: A17 -> GND
- U3 pad J8: A17 -> GND
- U3 pad M1: A17 -> GND
- U3 pad M9: A17 -> GND
- U3 pad P1: A17 -> GND
- U3 pad P9: A17 -> GND
- U3 pad T1: A17 -> GND
- U3 pad T9: A17 -> GND
- U4 pad 10: F10 -> +1V8
- U4 pad 14: A17 -> GND
- U4 pad 18: A17 -> +3V3
- U4 pad 19: A17 -> GND
- U4 pad 21: A17 -> GND
- U4 pad 3: A17 -> GND
- U4 pad 9: A17 -> GND
- U5 pad 10: A17 -> GND
- U5 pad 2: A17 -> GND
- U6 pad 2: A17 -> GND
- U6 pad 4: +5V -> SNS5V0
- U6 pad 5: +5V -> SNS5V0
- U7 pad 2: A17 -> GND
- U7 pad 4: +5V -> SNS5V0
- U7 pad 5: +5V -> SNS5V0
- U8 pad 3: F10 -> XADCGND
- U9 pad 2: A17 -> GND
- U9 pad 9: A17 -> GND
- Y4 pad 1: A17 -> +3V3
- Y4 pad 2: A17 -> GND
- Y4 pad 4: A17 -> +3V3
- Y5 pad 1: A17 -> +3V3
- Y5 pad 2: A17 -> GND
- Y5 pad 4: A17 -> +3V3
Other:
- board outline added: 110.4 x 87.4 mm
