File: A/CHIPKIT IO.kicad_sch (KiCad schematic)
At the start: 75 parts, among them J1 Conn_02x06_Top_Bottom, J2 Conn_02x08_Top_Bottom, J3 Conn_01x02, J4 Conn_02x08_Top_Bottom, J5 Conn_01x04, J6 Conn_02x03_Top_Bottom, J7 Conn_01x08

Commit message: Add files via upload
Updated
Parts:
- removed J1: Conn_02x06_Top_Bottom, Connector_PinSocket_2.54mm:PinSocket_2x06_P2.54mm_Vertical, symbol Connector_Generic:Conn_02x06_Top_Bottom
- removed J2, J4: Conn_02x08_Top_Bottom, Connector_PinSocket_2.54mm:PinSocket_2x08_P2.54mm_Vertical, symbol Connector_Generic:Conn_02x08_Top_Bottom
- removed J6: Conn_02x03_Top_Bottom, Connector_PinHeader_2.54mm:PinHeader_2x03_P2.54mm_Vertical, symbol Connector_Generic:Conn_02x03_Top_Bottom
- added J1: Conn_02x06_Odd_Even, Connector_PinSocket_2.54mm:PinSocket_2x06_P2.54mm_Vertical, symbol Connector_Generic:Conn_02x06_Odd_Even
- added J2, J4: Conn_02x08_Odd_Even, Connector_PinSocket_2.54mm:PinSocket_2x08_P2.54mm_Vertical, symbol Connector_Generic:Conn_02x08_Odd_Even
- added J6: Conn_02x03_Odd_Even, Connector_PinSocket_2.54mm:PinSocket_2x03_P2.54mm_Vertical, symbol Connector_Generic:Conn_02x03_Odd_Even
- C14, C15, C16, C17, C18, C19: footprint Capacitor_SMD:C_1206_3216Metric -> Capacitor_SMD:C_0805_2012Metric
- R155, R156, R59, R60, R61, R62, R63, R64, R65, R66, R67, R68, R69, R70, R71, R73, R75, R77, R79, R81: footprint Resistor_SMD:R_0201_0603Metric -> Resistor_SMD:R_0402_1005Metric
- R72, R74, R76, R78, R80, R82: footprint Resistor_SMD:R_1206_3216Metric -> Resistor_SMD:R_0402_1005Metric
Connections:
- net 0: now also J4.1 (Pin_1)
- net 1: now also J4.3 (Pin_3)
- net 10: now also J2.5 (Pin_5)
- net 11: now also J2.7 (Pin_7)
- net 12: now also J2.9 (Pin_9)
- net 13: now also J2.11 (Pin_11)
- net 2: now also J4.5 (Pin_5)
- net 26: now also J4.2 (Pin_2)
- net 27: now also J4.4 (Pin_4)
- net 28: now also J4.6 (Pin_6)
- net 29: now also J4.8 (Pin_8)
- net 3: now also J4.7 (Pin_7)
- net 30: now also J4.10 (Pin_10)
- net 31: now also J4.12 (Pin_12)
- net 32: now also J4.14 (Pin_14)
- net 33: now also J4.16 (Pin_16)
- net 34: now also J2.2 (Pin_2)
- net 35: now also J2.4 (Pin_4)
- net 36: now also J2.6 (Pin_6)
- net 37: now also J2.8 (Pin_8)
- net 38: now also J2.10 (Pin_10)
- net 39: now also J2.12 (Pin_12)
- net 4: now also J4.9 (Pin_9)
- net 40: now also J2.14 (Pin_14)
- net 41: now also J2.16 (Pin_16)
- net 5: now also J4.11 (Pin_11)
- net 6: now also J4.13 (Pin_13)
- net 7: now also J4.15 (Pin_15)
- net 8: now also J2.1 (Pin_1)
- net 9: now also J2.3 (Pin_3)
- net CK_A0: now also J1.1 (Pin_1)
- net CK_A1: now also J1.3 (Pin_3)
- net CK_A10: now also J1.10 (Pin_10)
- net CK_A11: now also J1.12 (Pin_12)
- net CK_A2: now also J1.5 (Pin_5)
- net CK_A3: now also J1.7 (Pin_7)
- net CK_A4: now also J1.9 (Pin_9)
- net CK_A5: now also J1.11 (Pin_11)
- net CK_A6: now also J1.2 (Pin_2)
- net CK_A7: now also J1.4 (Pin_4)
- net CK_A8: now also J1.6 (Pin_6)
- net CK_A9: now also J1.8 (Pin_8)
- net GND: now also J6.6 (Pin_6)
- net MISO: now reaches R39.2
- net MISO: now also J6.1 (Pin_1)
- net SCK: now reaches R40.2
- net SCK: now also J6.3 (Pin_3)
- net SS: now reaches R41.2
- net SS: now also J6.5 (Pin_5)
- net MOSI: now reaches R50.1
- net MOSI: now also J6.4 (Pin_4)
- net 14 renamed G
- net G: now also J2.13 (Pin_13)
- net 15 renamed A
- net A: now also J2.15 (Pin_15)
