File: A/FPGA BANK.kicad_sch (KiCad schematic)
At the start: 143 parts, among them J10 Conn_01x06, U1 XC7A100T-1CSG324C, U10 S25FL128SAGMFIR01, U13 TPD4E101DPWR, Y4 ASEM1-100.000MHZ-LC-T, Y5 ASEM1-100.000MHZ-LC-T

Commit message: Add files via upload
Updated
Parts:
- removed C186, C190, C192: 470nF, Capacitor_SMD:C_0805_2012Metric, symbol Device:C
- removed C187, C191: 47nF, Capacitor_SMD:C_0805_2012Metric, symbol Device:C
- removed C188: 47uF, Capacitor_SMD:C_0201_0603Metric, symbol Device:C
- removed C189, C193: 100uF, Capacitor_SMD:C_0805_2012Metric, symbol Device:C
- removed C202, C203: 100nF, Capacitor_SMD:C_0402_1005Metric, symbol Device:C
- removed U10: S25FL128SAGMFIR01, SO3016_SPA, symbol 2025-06-10_04-45-04:S25FL128SAGMFIR01
- added C60: 47uF, Capacitor_SMD:C_1210_3225Metric, symbol Device:C
- added C61, C63, C66, C67, C68, C69: 470nF, Capacitor_SMD:C_0603_1608Metric, symbol Device:C
- added C62, C65: 4.7uF, Capacitor_SMD:C_0805_2012Metric, symbol Device:C
- added C64, C70: 47nF, Capacitor_SMD:C_1206_3216Metric, symbol Device:C
- added JP2: Conn_01x02, Connector_PinHeader_1.00mm:PinHeader_1x02_P1.00mm_Vertical, symbol Connector_Generic:Conn_01x02
- added U10: S25FL128SAGMFI013, ul_S25FL128SAGMFI013:SO3016_SPA, symbol 2025-06-11_05-38-59:S25FL128SAGMFI013
- C105: footprint Capacitor_SMD:C_0402_1005Metric -> Capacitor_SMD:C_0603_1608Metric_Pad1.08x0.95mm_HandSolder
- C109: footprint Capacitor_SMD:C_1206_3216Metric -> Capacitor_SMD:C_0402_1005Metric
- C113, C136, C137, C138, C145, C146, C147, C153, C159, C167: value 100uF -> 47nF; footprint Capacitor_SMD:C_0805_2012Metric -> Capacitor_SMD:C_1206_3216Metric
- C114, C123, C124: value 4.7uF -> 47nF; footprint Capacitor_SMD:C_0402_1005Metric -> Capacitor_SMD:C_1206_3216Metric
- C115, C172, C173: footprint Capacitor_SMD:C_0402_1005Metric -> Capacitor_SMD:C_0805_2012Metric
- C116: value 470nF -> 100uF; footprint Capacitor_SMD:C_0805_2012Metric -> Capacitor_SMD:C_1206_3216Metric
- C117, C118: value 470nF -> 4.7uF
- C119, C176, C177, C184: footprint Capacitor_SMD:C_0805_2012Metric -> Capacitor_SMD:C_0603_1608Metric
- C120, C121, C122: value 47nF -> 470nF; footprint Capacitor_SMD:C_0805_2012Metric -> Capacitor_SMD:C_0603_1608Metric
- C125: value 470nF -> 47nF; footprint Capacitor_SMD:C_0805_2012Metric -> Capacitor_SMD:C_1206_3216Metric
- C126, C127, C128: value 470nF -> 10nF; footprint Capacitor_SMD:C_0805_2012Metric -> Capacitor_SMD:C_0201_0603Metric
- C129: value 47nF -> 100uF; footprint Capacitor_SMD:C_0805_2012Metric -> Capacitor_SMD:C_1206_3216Metric
- C130, C131: value 47nF -> 4.7uF
- C132, C133, C134, C135, C141, C142, C143, C144, C151, C152, C163, C164, C165, C166: value 100uF -> 470nF; footprint Capacitor_SMD:C_0805_2012Metric -> Capacitor_SMD:C_0603_1608Metric
- C139, C140, C149, C150, C161, C162, C170, C171: value 100uF -> 4.7uF
- C148, C168, C169: footprint Capacitor_SMD:C_0805_2012Metric -> Capacitor_SMD:C_1206_3216Metric
- C154, C156, C157, C158: value 100nF -> 47nF; footprint Capacitor_SMD:C_0402_1005Metric -> Capacitor_SMD:C_1206_3216Metric
- C155: value 100nF -> 470nF; footprint Capacitor_SMD:C_0402_1005Metric -> Capacitor_SMD:C_0603_1608Metric
- C160: value 100uF -> 47uF; footprint Capacitor_SMD:C_0805_2012Metric -> Capacitor_SMD:C_1210_3225Metric
- C174, C175, C182: value 4.7uF -> 470nF; footprint Capacitor_SMD:C_0402_1005Metric -> Capacitor_SMD:C_0603_1608Metric
- C178: value 470uF -> 470nF; footprint Capacitor_SMD:C_0805_2012Metric -> Capacitor_SMD:C_0603_1608Metric
- C179: value 470uF -> 10nF; footprint Capacitor_SMD:C_0805_2012Metric -> Capacitor_SMD:C_0201_0603Metric
- C180: value 470uF -> 100nF; footprint Capacitor_SMD:C_0805_2012Metric -> Capacitor_SMD:C_0201_0603Metric
- C181: value 4.7uF -> 100uF; footprint Capacitor_SMD:C_0402_1005Metric -> Capacitor_SMD:C_1206_3216Metric
- C183: value 470uF -> 47nF; footprint Capacitor_SMD:C_0805_2012Metric -> Capacitor_SMD:C_1206_3216Metric
- C185: value 470nF -> 100nF
- R123, R251, R252, R255, R256, R257, R308: footprint Resistor_SMD:R_1206_3216Metric -> Resistor_SMD:R_0402_1005Metric
- R140, R246, R247, R261, R262, R263, R264, R265, R266, R267, R268: footprint Resistor_SMD:R_0805_2012Metric -> Resistor_SMD:R_0402_1005Metric
- R248, R249: footprint Resistor_SMD:R_0201_0603Metric -> Resistor_SMD:R_0402_1005Metric
- R250, R253, R254, R271, R272, R273, R274, R275, R276, R296, R297: footprint Resistor_SMD:R_0603_1608Metric -> Resistor_SMD:R_0402_1005Metric
Connections:
- net SNSVCCINT_P is gone; now on net SNS5V0_P: R267.2
- net +1V0: now also C148.1, C149.1, C150.1, C151.1, C152.1, C153.1, C154.1, C155.1, C156.1, C157.1, C158.1, C159.1, C168.1, C169.1, C170.1, C171.1, C172.1, C173.1, C174.1, C175.1, C176.1, C177.1, C178.1, C181.1, C182.1, C183.1, C184.1
- net +1V8: now also C160.1, C161.1, C162.1, C163.1, C164.1, C165.1, C166.1, C167.1, C179.1, C180.1; no longer C181.1, C182.1, C183.1, C184.1, C185.1
- net +3V3: now also C185.1, C60.1, C61.1, C62.1, C63.1, C64.1, C65.1, C66.1, C67.1, C68.1, C69.1, C70.1, U10.2 (VCC); no longer BTN4.3, BTN4.4, BTN5.1, BTN5.2, C109.2, C113.2, C114.2, C115.2, C116.1, C116.2, C117.1, C117.2, C118.1, C118.2, C119.1, C119.2, C120.1, C120.2, C121.1, C121.2, C122.1, C122.2, C123.1, C123.2, C124.1, C124.2, C125.1, C125.2, C126.1, C126.2, C127.1, C127.2, C128.1, C128.2, C129.2, C130.2, C131.2, C132.2, C133.2, C134.2, C135.2, C136.2, C137.2, C138.2, C139.2, C140.2, C141.2, C142.2, C143.2, C144.2, C145.2, C146.2, C147.2, C148.1, C148.2, C149.1, C149.2, C150.1, C150.2, C151.1, C151.2, C152.1, C152.2, C153.1, C153.2, C154.1, C154.2, C155.1, C155.2, C156.1, C156.2, C157.1, C157.2, C158.1, C158.2, C159.1, C159.2, C160.1, C160.2, C161.1, C161.2, C162.1, C162.2, C163.1, C163.2, C164.1, C164.2, C165.1, C165.2, C166.1, C166.2, C167.1, C167.2, C168.1, C168.2, C169.1, C169.2, C170.1, C170.2, C171.1, C171.2, C172.1, C172.2, C173.1, C173.2, C174.1, C174.2, C175.1, C175.2, C176.1, C176.2, C177.1, C177.2, C178.1, C178.2, C179.1, C179.2, C180.1, C180.2, C181.2, C182.2, C183.2, C184.2, C185.2, C204.2, J10.5 (Pin_5), JP1.2 (Pin_2), LD8.1 (K), R248.2, R256.1, R308.1, U1.A12 (GND), U1.A2 (GND), U1.B15 (GND), U1.B5 (GND), U1.C18 (GND), U1.C8 (GND), U1.D1 (GND), U1.D11 (GND), U1.E14 (GND), U1.E4 (GND), U1.F11 (GND), U1.F17 (GND), U1.F7 (GND), U1.F9 (GND), U1.G10 (GND), U1.G12 (GND), U1.G8 (GND), U1.H11 (GND), U1.H13 (GND), U1.H3 (GND), U1.H7 (GND), U1.H9 (GNDADC_0), U1.J12 (GND), U1.J16 (GND), U1.J6 (GND), U1.J8 (GND), U1.K11 (GND), U1.K7 (GND), U1.L10 (DXP_0), U1.L12 (GND), U1.L2 (GND), U1.L8 (GND), U1.L9 (DXN_0), U1.M11 (GND), U1.M15 (GND), U1.M5 (GND), U1.M7 (GND), U1.M9 (GND), U1.N10 (GND), U1.N12 (GND), U1.N18 (GND), U1.N8 (GND), U1.P1 (GND), U1.P6 (VCCO_34), U1.R14 (GND), U1.R4 (GND), U1.T17 (GND), U1.T2 (VCCO_34), U1.T7 (GND), U1.U10 (GND), U1.U5 (VCCO_34), U1.V13 (GND), U1.V3 (GND), U1.V8 (VCCO_34), U13.5, Y4.2 (GND), Y5.2 (GND)
- net CK_RST: now also C185.2, JP2.1 (Pin_1)
- net QSPI_CS: now also U10.7 (*CS)
- net QSPI_SCK: now also U10.16 (SCK)
- net SNS5V0_P: no longer R264.2
- net at R259.1: now also U10.1 (*HOLD/IO3)
- net at R260.2: now also U10.8 (SO/IO1)
- net at R123.2: now also U10.15 (SI/IO0)
- net at R258.1: now also U10.9 (*WP/IO2)
- net SNSVCCINT_N renamed SNS5V0_N
- net SNS5V0_N: now also R264.2
- net SW0 renamed S1
- net SW1 renamed S2
- net SW2 renamed S3
- net SW3 renamed S4
- new net DDRVCC: C116.1, C117.1, C118.1, C119.1, C120.1, C121.1, C122.1, C123.1, C124.1, C125.1, C126.1, C127.1, C128.1, U1.P6 (VCCO_34), U1.T2 (VCCO_34), U1.U5 (VCCO_34), U1.V8 (VCCO_34)
- new net GND: BTN4.3, BTN4.4, BTN5.1, BTN5.2, C109.2, C113.2, C114.2, C115.2, C116.2, C117.2, C118.2, C119.2, C120.2, C121.2, C122.2, C123.2, C124.2, C125.2, C126.2, C127.2, C128.2, C129.2, C130.2, C131.2, C132.2, C133.2, C134.2, C135.2, C136.2, C137.2, C138.2, C139.2, C140.2, C141.2, C142.2, C143.2, C144.2, C145.2, C146.2, C147.2, C148.2, C149.2, C150.2, C151.2, C152.2, C153.2, C154.2, C155.2, C156.2, C157.2, C158.2, C159.2, C160.2, C161.2, C162.2, C163.2, C164.2, C165.2, C166.2, C167.2, C168.2, C169.2, C170.2, C171.2, C172.2, C173.2, C174.2, C175.2, C176.2, C177.2, C178.2, C179.2, C180.2, C181.2, C182.2, C183.2, C184.2, C204.2, C60.2, C61.2, C62.2, C63.2, C64.2, C65.2, C66.2, C67.2, C68.2, C69.2, C70.2, J10.5 (Pin_5), JP1.2 (Pin_2), JP2.2 (Pin_2), LD8.1 (K), R248.2, R256.1, R308.1, U1.A12 (GND), U1.A2 (GND), U1.B15 (GND), U1.B5 (GND), U1.C18 (GND), U1.C8 (GND), U1.D1 (GND), U1.D11 (GND), U1.E14 (GND), U1.E4 (GND), U1.F11 (GND), U1.F17 (GND), U1.F7 (GND), U1.F9 (GND), U1.G10 (GND), U1.G12 (GND), U1.G8 (GND), U1.H11 (GND), U1.H13 (GND), U1.H3 (GND), U1.H7 (GND), U1.H9 (GNDADC_0), U1.J12 (GND), U1.J16 (GND), U1.J6 (GND), U1.J8 (GND), U1.K11 (GND), U1.K7 (GND), U1.L10 (DXP_0), U1.L12 (GND), U1.L2 (GND), U1.L8 (GND), U1.L9 (DXN_0), U1.M11 (GND), U1.M15 (GND), U1.M5 (GND), U1.M7 (GND), U1.M9 (GND), U1.N10 (GND), U1.N12 (GND), U1.N18 (GND), U1.N8 (GND), U1.P1 (GND), U1.R14 (GND), U1.R4 (GND), U1.T17 (GND), U1.T7 (GND), U1.U10 (GND), U1.V13 (GND), U1.V3 (GND), U10.10 (VSS), U13.5, Y4.2 (GND), Y5.2 (GND)
- no-connect marks 5 -> 7
Other:
- moved on the sheet: R123, R258, R259, R260
