File: A/LED.kicad_sch (KiCad schematic)
At the start: 54 parts, among them Q10 DMMT5401-7-F, Q11 DMMT5401-7-F, Q12 DMMT5401-7-F, Q7 DMMT5401-7-F, Q8 DMMT5401-7-F, Q9 DMMT5401-7-F

Commit message: Add files via upload
Updated
Parts:
- removed LD0, LD1, LD2, LD3: 19-337/R6GHBHC-A01/2T, 19-337_R6GHBHC-A01_2T:LED_19-337_R6GHBHC-A01_2T, symbol LED-TRISTATE:19-337_R6GHBHC-A01_2T
- added D1, D2, D3, D4: 19-337_R6GHBHC-A01_2T, 19-337_R6GHBHC-A01_2T:LED_19-337_R6GHBHC-A01_2T, symbol 19-337_R6GHBHC-A01_2T:19-337_R6GHBHC-A01_2T
- R166, R173, R174, R175, R178, R179, R180, R181, R182, R183, R186, R187, R188, R189, R190, R191, R192, R195, R196, R197, R198, R199, R200, R201, R204, R205, R206, R207, R208, R209, R37, R38: footprint Resistor_SMD:R_0201_0603Metric -> Resistor_SMD:R_0402_1005Metric
- R176, R184, R193, R202: footprint Resistor_SMD:R_2512_6332Metric -> Resistor_SMD:R_0402_1005Metric
- R177, R185, R194, R203: footprint Resistor_SMD:R_0805_2012Metric -> Resistor_SMD:R_0402_1005Metric
Connections:
- net at Q12.4: now also D4.6
- net at Q10.4: now also D4.4
- net at R192.2: now also D3.1
- net at Q8.4: now also D2.5
- net at R193.2: now also D3.2
- net at R176.2: now also D1.2
- net at R203.2: now also D4.3
- net at R166.2: now also D2.1
- net at R184.2: now also D2.2
- net at R185.2: now also D2.3
- net at Q7.4: now also D2.4
- net at Q9.4: now also D2.6
- net at Q10.1: now also D3.4
- net at R177.2: now also D1.3
- net at R175.2: now also D1.1
- net at R194.2: now also D3.3
- net at Q12.1: now also D3.6
- net at Q7.1: now also D1.4
- net at Q8.1: now also D1.5
- net at Q11.1: now also D3.5
- net at R201.2: now also D4.1
- net at R202.2: now also D4.2
- net at Q11.4: now also D4.5
- net at Q9.1: now also D1.6
Other:
- moved on the sheet: R166, R175, R176, R177, R184, R185, R192, R193, R194, R201, R202, R203
