File: A/USB,UART.kicad_sch (KiCad schematic)
At the start: 67 parts, among them J12 USB_B, J13 Conn_01x08_Pin, J14 Conn_01x02, J15 Conn_01x02, U11 FT2232HL-REEL, U12 93LC56BT-I_OT, U14 SN74LVC126APW, Y3 25MHz

Commit message: Add files via upload
Updated
Parts:
- added D5, D6: D_TVS, Diode_SMD:D_0603_1608Metric, symbol Device:D_TVS
- R111, R112, R113, R114, R115, R116, R117, R118, R119, R120, R121, R122, R277, R278, R279, R280, R281, R282, R283, R284, R285, R286, R287, R288, R289, R290, R291, R292, R293, R294, R298, R299, R300, R301, R302, R303, R304, R305, R306, R307: footprint Resistor_SMD:R_1206_3216Metric -> Resistor_SMD:R_0402_1005Metric
Connections:
- net GND: now also D5.1 (A1), D6.1 (A1)
- net USB_D+: now also D6.2 (A2)
- net USB_D-: now also D5.2 (A2)
Other:
- moved on the sheet: C201, R277, R278, R279, R280
