File: A/connector.kicad_sch (KiCad schematic)
At the start: 56 parts, among them SW0 EG1218, SW1 EG1218, SW2 EG1218, SW3 EG1218

Commit message: Add files via upload
Updated
Parts:
- removed SW0, SW1, SW2, SW3: EG1218, EG1218:SW_EG1218, symbol EG1218:EG1218
- added S1, S2, S3, S4: EG1218, EG1218:SW_EG1218, symbol EG1218:EG1218
- R25, R26, R27, R28, R29, R30, R31, R32, R33, R34, R35, R36: footprint Resistor_SMD:R_0805_2012Metric -> Resistor_SMD:R_0402_1005Metric
Connections:
- net +3V3: now also S1.1, S2.1, S3.1, S4.1
- net GND: now also S1.3, S2.3, S3.3, S4.3
- net at R36.1: now also S4.2
- net at R33.1: now also S1.2
- net at R35.1: now also S3.2
- net at R34.1: now also S2.2
- net SW0 renamed S1
- net SW1 renamed S2
- net SW2 renamed S3
- net SW3 renamed S4
