File: A/power regulation.kicad_sch (KiCad schematic)
At the start: 16 parts, among them J9 Conn_01x06, U4 MP5470GL-0000-Z

Commit message: Add files via upload
Updated
Parts:
- R108, R109: footprint Resistor_SMD:R_0201_0603Metric -> Resistor_SMD:R_0402_1005Metric
Changed lines of the file:
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@@
 			)
 		)
-		(property "Footprint" "Resistor_SMD:R_0201_0603Metric"
+		(property "Footprint" "Resistor_SMD:R_0402_1005Metric"
 			(at 171.45 114.3 0)
 			(effects
@@
 			)
 		)
-		(property "Footprint" "Resistor_SMD:R_0201_0603Metric"
+		(property "Footprint" "Resistor_SMD:R_0402_1005Metric"
 			(at 171.45 111.76 0)
 			(effects
