File: A/power regulations_sch.kicad_sch (KiCad schematic)
At the start: 80 parts, among them IC1 NCP380 ADJ, J11 DCJ200-10-A-XX-K_REVA, Q1 CSD25310Q2, Q2 BF459, Q3 BF459, Q4 BF459, Q5 BF459, Q6 BF459, U5 MP8756GD-Z, U6 INA199A1DCKR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

Commit message: Add files via upload
Updated
Parts:
- removed Q3, Q4, Q5, Q6: BF459, Package_TO_SOT_THT:TO-126-3_Vertical, symbol Transistor_BJT:BF459
- added Q3, Q4: DMMT5401-7-F, DMMT5401-7-F:SOT95P285X140-6N, symbol DMMT5401-7-F:DMMT5401-7-F
- C100, C102: value 470uF -> 470nF; footprint Capacitor_SMD:C_1812_4532Metric -> Capacitor_SMD:C_0603_1608Metric
- C83, C84, C85, C88, C89: footprint Capacitor_SMD:C_0201_0603Metric -> Capacitor_SMD:C_0402_1005Metric
- R125, R138, R17, R21, R23, R24: footprint Resistor_SMD:R_1206_3216Metric -> Resistor_SMD:R_0402_1005Metric
- R129, R132, R136, R158, R167, R168, R169, R172, R18, R19, R22: footprint Resistor_SMD:R_0201_0603Metric -> Resistor_SMD:R_0402_1005Metric
- R131, R135, R157, R160, R162, R164, R165, R170, R171: footprint Resistor_SMD:R_0805_2012Metric -> Resistor_SMD:R_0402_1005Metric
Connections:
- net +5V: no longer U6.4 (IN+), U6.5 (IN-), U7.4 (IN+), U7.5 (IN-)
- net GND: now also Q3.5, Q3.6, Q4.1, Q4.4
- net PGVREG5V0: now also Q4.2, Q4.3
- net at R161.1: now also Q4.6
- net at R171.1: now also Q3.4
- net at R172.1: now also Q3.1, Q3.3
- net at R19.1: now also Q3.2
- net at R165.2, R167.1: now also Q4.5
- new net SNS5V0: U6.4 (IN+), U6.5 (IN-), U7.4 (IN+), U7.5 (IN-)
